File: Kicad/Catpucciano.kicad_sch (KiCad schematic)
At the start: 57 parts, among them SW1 RSW, SW2 PSW

Commit message: Reorganized Files
Parts:
- removed H1: BAT+, symbol ScottoKeebs:Placeholder_Mounting_Hole
- removed H2: BATGND, symbol ScottoKeebs:Placeholder_Mounting_Hole
- removed SW2: PSW, symbol Switch:SW_Push_SPDT
- added J1: Conn_01x02, Connector_JST:JST_EH_S2B-EH_1x02_P2.50mm_Horizontal, symbol Connector_Generic:Conn_01x02
- added SW3: Switch, ScottoKeebs_Components:Switch_MSK12C02, symbol ScottoKeebs:Placeholder_Switch
- D1, D10, D11, D12, D13, D14, D15, D16, D17, D18, D19, D2, D20, D21, D22, D23, D24, D25, D26, D3, D4, D5, D6, D7, D8, D9: footprint (none) -> ScottoKeebs_Components:Diode_SOD-123
- S1, S10, S11, S12, S13, S14, S15, S16, S17, S18, S19, S2, S20, S21, S22, S23, S24, S25, S26, S3, S4, S5, S6, S7, S8, S9: footprint (none) -> ScottoKeebs_Hotswap:Hotswap_Choc_V1_1.00u
- SW1: footprint (none) -> Button_Switch_SMD:Panasonic_EVQPUL_EVQPUC
- xiao-ble1: renamed from xiao-ble; footprint (none) -> test:xiao-ble-tht
Connections:
- net BAT+: now also SW3.1
- net GND: now also J1.1 (Pin_1)
- net VBAT: now also J1.2 (Pin_2), SW3.2
Other:
- note added: "BATTERY (JST Connector)"
- note removed: "BATTERY"
